Commit message: Scale large courier to 3x the Parrot
- courier_large.urdf.xacro: scale 1.5 -> 3.0; body box now derived from
  scale (1.0 x 1.14 x 0.27 m), mass unchanged at 1.006 kg. IMU z 0.18,
  lidar z 0.35, camera (0.30, 0, -0.30) to stay clear of the body.
- nav2_params_parrot2_large.yaml: footprint +/-0.55 x +/-0.62 m,
  inflation radius 1.1 m.

Co-Authored-By: Claude Opus 5.5 <noreply@anthropic.com>

File: urdf_parrot/courier_large.urdf.xacro (robot description, xacro)
@@ -1,4 +1,4 @@
 <?xml version="1.0" ?>
-<!-- Large courier variant of parrot.urdf.xacro: 1.5x the size, 2x the mass.
+<!-- Large courier variant of parrot.urdf.xacro: 3x the size, 2x the mass.
      Uses the same parrot.gazebo.xacro, so plugins and Gazebo topics
      (/model/<gz_model_name>/...) are identical to the original Parrot. -->
@@ -13,12 +13,12 @@
   <xacro:property name="r200_cam_depth_offset" value="0.01"/>
   <!-- Size and mass relative to the original Parrot (0.503 kg). -->
-  <xacro:property name="scale" value="1.5"/>
+  <xacro:property name="scale" value="3.0"/>
   <xacro:property name="body_mass" value="${0.503 * 2.0}"/>
   <!-- Body bounding box including propellers. The original is about
-       0.33 x 0.38 x 0.09 m (hull.dae is 0.18 x 0.22 x 0.07 m with a 1.223x
-       node scale, plus the propellers), so 1.5x gives roughly the box below. -->
-  <xacro:property name="body_x" value="0.50"/>
-  <xacro:property name="body_y" value="0.57"/>
-  <xacro:property name="body_z" value="0.14"/>
+       0.333 x 0.38 x 0.09 m (hull.dae is 0.18 x 0.22 x 0.07 m with a 1.223x
+       node scale, plus the propellers); at 3x that is 1.0 x 1.14 x 0.27 m. -->
+  <xacro:property name="body_x" value="${0.333 * scale}"/>
+  <xacro:property name="body_y" value="${0.38 * scale}"/>
+  <xacro:property name="body_z" value="${0.09 * scale}"/>
   <!-- Main link -->
   <link name="${prefix}base_link">
@@ -68,9 +68,9 @@
   </link>
   <!-- Sensors moved outward so they sit clear of the larger body
-       (top of body ~ +0.06 m, bottom ~ -0.08 m). -->
+       (top of body ~ +0.12 m, bottom ~ -0.15 m). -->
   <joint name="${prefix}imu_joint" type="fixed">
     <parent link="${prefix}base_link"/>
     <child link="${prefix}imu_link"/>
-    <origin xyz="0.0 0 0.10" rpy="0 0 0"/> <!-- original: 0.068 -->
+    <origin xyz="0.0 0 0.18" rpy="0 0 0"/> <!-- original: 0.068 -->
   </joint>
   <link name="${prefix}imu_link"/>
@@ -78,5 +78,5 @@
     <parent link="${prefix}base_link"/>
     <child link="${prefix}base_scan"/>
-    <origin xyz="0 0 0.30" rpy="0 0 0"/> <!-- original: 0.2 -->
+    <origin xyz="0 0 0.35" rpy="0 0 0"/> <!-- original: 0.2 -->
   </joint>
   <link name="${prefix}base_scan">
@@ -97,5 +97,5 @@
   </link>
   <joint name="${prefix}camera_joint" type="fixed">
-    <origin xyz="0.25 0.0 -0.25" rpy="0 1.5708 0"/> <!-- original: 0.15 0.0 -0.2 -->
+    <origin xyz="0.30 0.0 -0.30" rpy="0 1.5708 0"/> <!-- original: 0.15 0.0 -0.2 -->
     <parent link="${prefix}base_link"/>
     <child link="${prefix}camera_link"/>
